Commit message: Change directory structure. Added namespace to have the opportunity to use multiple robots.

File: urdf/bringups/ur10_on_stand.urdf.xacro (robot description, xacro)
@@ -1,14 +1,14 @@
 <?xml version="1.0"?>
-<robot xmlns:xacro="http://wiki.ros.org/xacro" name="ur10e">
+<robot xmlns:xacro="http://wiki.ros.org/xacro" name="ur10">
   <!-- resolve prefix variable (useful for multi robot) -->
-  <xacro:include filename="$(find chargepal_description)/urdf/prefix.urdf.xacro" />
+  <xacro:include filename="$(find chargepal_description)/urdf/utils/prefix.urdf.xacro" />
   <!-- arm base, orange block/mount for ur5 or ur10 arm -->
-  <xacro:include filename="$(find chargepal_description)/urdf/stand.urdf.xacro" />
-  <!-- ur10e arm without ros control-->
-  <xacro:include filename="$(find chargepal_description)/urdf/ur10e.urdf.xacro" />
+  <xacro:include filename="$(find chargepal_description)/urdf/environment/stand.urdf.xacro" />
+  <!-- ur10 arm without ros control-->
+  <xacro:include filename="$(find chargepal_description)/urdf/ur_arm/ur10.urdf.xacro" />
   <!-- attach "arm" and "arm base" -->
   <joint name="${prefix}arm_base_to_arm" type="fixed">
     <parent link="${prefix}arm_base" />
-    <child link="${prefix}ur10e_base_link" />
+    <child link="${prefix}ur10_base_link" />
     <origin xyz="0 0 1.0" rpy="0 0 0" />
   </joint>
@@ -16,5 +16,5 @@
   <gazebo>
     <plugin name="ros_control" filename="libgazebo_ros_control.so">
-       <robotNamespace>/ur10e</robotNamespace>
+       <robotNamespace>/ur10</robotNamespace>
     </plugin>
   </gazebo>

File: urdf/bringups/ur5_on_stand.urdf.xacro (robot description, xacro)
@@ -1,14 +1,14 @@
 <?xml version="1.0"?>
-<robot xmlns:xacro="http://wiki.ros.org/xacro" name="ur10">
+<robot xmlns:xacro="http://wiki.ros.org/xacro" name="ur5">
   <!-- resolve prefix variable (useful for multi robot) -->
-  <xacro:include filename="$(find chargepal_description)/urdf/prefix.urdf.xacro" />
+  <xacro:include filename="$(find chargepal_description)/urdf/utils/prefix.urdf.xacro" />
   <!-- arm base, orange block/mount for ur5 or ur10 arm -->
-  <xacro:include filename="$(find chargepal_description)/urdf/stand.urdf.xacro" />
-  <!-- ur10 arm without ros control-->
-  <xacro:include filename="$(find chargepal_description)/urdf/ur10.urdf.xacro" />
+  <xacro:include filename="$(find chargepal_description)/urdf/environment/stand.urdf.xacro" />
+  <!-- ur5 arm without ros control-->
+  <xacro:include filename="$(find chargepal_description)/urdf/ur_arm/ur5.urdf.xacro" />
   <!-- attach "arm" and "arm base" -->
   <joint name="${prefix}arm_base_to_arm" type="fixed">
     <parent link="${prefix}arm_base" />
-    <child link="${prefix}ur10_base_link" />
+    <child link="${prefix}ur5_base_link" />
     <origin xyz="0 0 1.0" rpy="0 0 0" />
   </joint>
@@ -16,5 +16,5 @@
   <gazebo>
     <plugin name="ros_control" filename="libgazebo_ros_control.so">
-       <robotNamespace>/ur10</robotNamespace>
+       <robotNamespace>/ur5</robotNamespace>
     </plugin>
   </gazebo>

File: urdf/calibrated/calib_ur5.urdf.xacro (robot description, xacro)
@@ -3,5 +3,5 @@
   <!--calibrated and joint limited ur5 without ros control-->
   <!-- resolve prefix variable (useful for multi robot) -->
-  <xacro:include filename="$(find chargepal_description)/urdf/prefix.urdf.xacro" />
+  <xacro:include filename="$(find chargepal_description)/urdf/utils/prefix.urdf.xacro" />
   <!-- ################################################################### -->
   <!-- ur5 arm -->

File: urdf/environment/stand.urdf.xacro (robot description, xacro)
@@ -3,12 +3,12 @@
   <!-- arm base, orange block/mount for ur5 or ur10 arm -->
   <!-- resolve prefix variable (useful for multi robot) -->
-  <xacro:include filename="$(find chargepal_description)/urdf/prefix.urdf.xacro" />
+  <xacro:include filename="$(find chargepal_description)/urdf/utils/prefix.urdf.xacro" />
   <!-- ################################################################### -->
   <!-- "arm base" : make box to elevate the robot arm -->
   <!-- fix arm base, so that it does not fall -->
-  <link name="world"/>
-  <joint name="world_to_robot" type="fixed">
-    <parent link="world"/>
-    <child link="arm_base"/>
+  <link name="${prefix}world"/>
+  <joint name="${prefix}world_to_robot" type="fixed">
+    <parent link="${prefix}world"/>
+    <child link="${prefix}arm_base"/>
     <origin xyz="0 0 0" rpy="0 0 0"/>
   </joint>
@@ -37,5 +37,5 @@
     </inertial>
   </link>
-  <gazebo reference="arm_base">
+  <gazebo reference="${prefix}arm_base">
     <material>Gazebo/Orange</material> <!-- gazebo will read this color -->
   </gazebo>

File: urdf/ur_arm/ur10.urdf.xacro (robot description, xacro)
@@ -3,5 +3,5 @@
   <!--ur10 without ros control-->
   <!-- resolve prefix variable (useful for multi robot) -->
-  <xacro:include filename="$(find chargepal_description)/urdf/prefix.urdf.xacro" />
+  <xacro:include filename="$(find chargepal_description)/urdf/utils/prefix.urdf.xacro" />
   <!-- ################################################################### -->
   <!-- ur10 arm -->

File: urdf/ur_arm/ur10e.urdf.xacro (robot description, xacro)
@@ -3,5 +3,5 @@
   <!--ur10e without ros control-->
   <!-- resolve prefix variable (useful for multi robot) -->
-  <xacro:include filename="$(find chargepal_description)/urdf/prefix.urdf.xacro" />
+  <xacro:include filename="$(find chargepal_description)/urdf/utils/prefix.urdf.xacro" />
   <!-- ################################################################### -->
   <!-- ur10e arm -->

File: urdf/ur_arm/ur5.urdf.xacro (robot description, xacro)
@@ -3,5 +3,5 @@
   <!--ur5 without ros control-->
   <!-- resolve prefix variable (useful for multi robot) -->
-  <xacro:include filename="$(find chargepal_description)/urdf/prefix.urdf.xacro" />
+  <xacro:include filename="$(find chargepal_description)/urdf/utils/prefix.urdf.xacro" />
   <!-- ################################################################### -->
   <!-- ur5 arm -->

Commit message: Add a first primitive chargepal robot with a static platform and a robotiq 140 gripper.

File: urdf/bringups/ur10_on_stand.urdf.xacro (robot description, xacro)
@@ -14,8 +14,5 @@
   </joint>
   <!-- ros control -->
-  <gazebo>
-    <plugin name="ros_control" filename="libgazebo_ros_control.so">
-       <robotNamespace>/ur10</robotNamespace>
-    </plugin>
-  </gazebo>
+  <xacro:include filename="$(find chargepal_description)/urdf/utils/common.gazebo.xacro" />
+  <xacro:controller_plugin_gazebo robot_namespace=""/>
 </robot>

File: urdf/bringups/ur10e_on_stand.urdf.xacro (robot description, xacro)
@@ -14,8 +14,5 @@
   </joint>
   <!-- ros control -->
-  <gazebo>
-    <plugin name="ros_control" filename="libgazebo_ros_control.so">
-       <robotNamespace>/ur10e</robotNamespace>
-    </plugin>
-  </gazebo>
+  <xacro:include filename="$(find chargepal_description)/urdf/utils/common.gazebo.xacro" />
+  <xacro:controller_plugin_gazebo robot_namespace=""/>
 </robot>

File: urdf/bringups/ur5_on_stand.urdf.xacro (robot description, xacro)
@@ -14,8 +14,5 @@
   </joint>
   <!-- ros control -->
-  <gazebo>
-    <plugin name="ros_control" filename="libgazebo_ros_control.so">
-       <robotNamespace>/ur5</robotNamespace>
-    </plugin>
-  </gazebo>
+  <xacro:include filename="$(find chargepal_description)/urdf/utils/common.gazebo.xacro" />
+  <xacro:controller_plugin_gazebo robot_namespace=""/>
 </robot>

File: urdf/environment/stand.urdf.xacro (robot description, xacro)
@@ -7,7 +7,7 @@
   <!-- "arm base" : make box to elevate the robot arm -->
   <!-- fix arm base, so that it does not fall -->
-  <link name="${prefix}world"/>
+  <link name="world"/>
   <joint name="${prefix}world_to_robot" type="fixed">
-    <parent link="${prefix}world"/>
+    <parent link="world"/>
     <child link="${prefix}arm_base"/>
     <origin xyz="0 0 0" rpy="0 0 0"/>
