Commit message: Add new testbed descriptions

File: urdf/bringups/chargepal_testbed_fix_rod.urdf.xacro (robot description, xacro)
@@ -75,4 +75,45 @@
     <origin xyz="0.0 0.0 0.0" rpy="0.0 0.0 0.0" />
   </joint>
+  <!-- ############### FIX ROD ################ -->
+  <xacro:property name="ROD_DIAMETER" value="34.5"/>
+  <xacro:include filename="$(find chargepal_tools)/urdf/rod.urdf.xacro" />
+  <xacro:rod_tool parent="${prefix}ft_sensor_wrench" prefix="${prefix}" diameter="${ROD_DIAMETER}" />
+  <!-- Add three (for each axis) additional virtual frames for reward calculation -->
+  <xacro:chargepal_virtual_joint
+    joint_name="${prefix}virt_tool_frame_x_joint"
+    type="fixed"
+    parent="${prefix}plug_reference_frame"
+    child="${prefix}virt_tool_frame_x"
+    joint_axis_xyz="0 0 0"
+    joint_origin_xyz="1 0 0"
+    joint_origin_rpy="0 0 0"
+    joint_lower_limit="0"
+    joint_upper_limit="0"
+  />
+  <xacro:chargepal_virtual_link link_name="${prefix}virt_tool_frame_x" />
+  <xacro:chargepal_virtual_joint
+    joint_name="${prefix}virt_tool_frame_y_joint"
+    type="fixed"
+    parent="${prefix}plug_reference_frame"
+    child="${prefix}virt_tool_frame_y"
+    joint_axis_xyz="0 0 0"
+    joint_origin_xyz="0 1 0"
+    joint_origin_rpy="0 0 0"
+    joint_lower_limit="0"
+    joint_upper_limit="0"
+  />
+  <xacro:chargepal_virtual_link link_name="${prefix}virt_tool_frame_y" />
+  <xacro:chargepal_virtual_joint
+    joint_name="${prefix}virt_tool_frame_z_joint"
+    type="fixed"
+    parent="${prefix}plug_reference_frame"
+    child="${prefix}virt_tool_frame_z"
+    joint_axis_xyz="0 0 0"
+    joint_origin_xyz="0 0 1"
+    joint_origin_rpy="0 0 0"
+    joint_lower_limit="0"
+    joint_upper_limit="0"
+  />
+  <xacro:chargepal_virtual_link link_name="${prefix}virt_tool_frame_z" />
   <!-- ################ GAZEBO ################ -->
   <!-- Common -->

File: urdf/ur_arm/ur10e.urdf.xacro (robot description, xacro)
@@ -7,5 +7,5 @@
   <!-- ur10e arm -->
   <xacro:include filename="$(find ur_description)/urdf/inc/ur10e_macro.xacro" />
-  <xacro:ur10e_robot prefix="${prefix}ur10e_" />
+  <xacro:ur10e_robot prefix="${prefix}" />
   <!-- ################################################################### -->
 </robot>
