Commit message: Add testbed description with Robot configuration like in the CIC building

File: urdf/bringups/chargepal_testbed_cic.urdf.xacro (robot description, xacro)
@@ -8,5 +8,5 @@
   <xacro:include filename="$(find chargepal_description)/urdf/utils/prefix.urdf.xacro" />
   <!-- ############### Table ################ -->
-  <xacro:include filename="$(find chargepal_description)/urdf/environment/testbed_table.urdf.xacro"/>
+  <xacro:include filename="$(find chargepal_description)/urdf/environment/testbed_table_cic.urdf.xacro"/>
   <!-- platform arm joint -->
   <joint name="${prefix}testbed_to_ur10e" type="fixed">
@@ -76,7 +76,6 @@
   </joint>
   <!-- ############### FIX ROD ################ -->
-  <xacro:property name="ROD_DIAMETER" value="34.5"/>
-  <xacro:include filename="$(find chargepal_tools)/urdf/rod.urdf.xacro" />
-  <xacro:rod_tool parent="${prefix}ft_sensor_wrench" prefix="${prefix}" diameter="${ROD_DIAMETER}" />
+  <xacro:include filename="$(find chargepal_description)/urdf/tools/tdt_plug.urdf.xacro" />
+  <xacro:tdt_plug parent="${prefix}ft_sensor_wrench" prefix="${prefix}" />
   <!-- ################ GAZEBO ################ -->
   <!-- Common -->
