Commit message: Change name pillar to adapter station

File: urdf/environment/primitive_adapter_station.urdf.xacro (robot description, xacro)
@@ -1,10 +1,10 @@
 <?xml version="1.0"?>
-<robot xmlns:xacro="http://ros.org/wiki/xacro" name="primitive_pillar">
+<robot xmlns:xacro="http://ros.org/wiki/xacro" name="primitive_adapter_station">
   <xacro:include filename="$(find chargepal_description)/urdf/utils/common_properties.urdf.xacro" />
   <!-- object properties -->
-  <xacro:property name="pillar_width" value="0.25" />
+  <xacro:property name="station_width" value="0.25" />
   <xacro:property name="socket_size" value="0.07" />
   <xacro:property name="socket_height" value="1.20" />
-  <xacro:property name="panel_thickness" value="${0.5*(pillar_width-socket_size)}" />
+  <xacro:property name="panel_thickness" value="${0.5*(station_width-socket_size)}" />
   <!-- start kinematic chain -->
   <link name="world" />
@@ -15,5 +15,5 @@
   </joint>
   <link name="low_body_link">
-    <xacro:box_inertial_ x="${pillar_width}" y="${pillar_width}" z="${socket_height - 0.5*socket_size}" mass="50.0">
+    <xacro:box_inertial_ x="${station_width}" y="${station_width}" z="${socket_height - 0.5*socket_size}" mass="50.0">
       <origin xyz="0 0 0" rpy="0 0 0" />
     </xacro:box_inertial_>
@@ -21,5 +21,5 @@
       <orign rpy="0.0 0.0 0.0" xyz="0.0 0.0 0.0" />
       <geometry>
-        <box size="${pillar_width} ${pillar_width} ${socket_height - 0.5*socket_size}" />
+        <box size="${station_width} ${station_width} ${socket_height - 0.5*socket_size}" />
       </geometry>
     </visual>
@@ -27,5 +27,5 @@
       <orign rpy="0.0 0.0 0.0" xyz="0.0 0.0 0.0" />
       <geometry>
-        <box size="${pillar_width} ${pillar_width} ${socket_height - 0.5*socket_size}" />
+        <box size="${station_width} ${station_width} ${socket_height - 0.5*socket_size}" />
       </geometry>
     </collision>
@@ -34,8 +34,8 @@
     <parent link="low_body_link" />
     <child link="left_panel_link" />
-    <origin rpy="0.0 0.0 0.0" xyz="${-0.25*(pillar_width+socket_size)} 0.0 ${0.5*socket_height + 0.25*socket_size}" />
+    <origin rpy="0.0 0.0 0.0" xyz="${-0.25*(station_width+socket_size)} 0.0 ${0.5*socket_height + 0.25*socket_size}" />
   </joint>
   <link name="left_panel_link">
-    <xacro:box_inertial_ x="${panel_thickness}" y="${pillar_width}" z="${socket_size}" mass="5.0">
+    <xacro:box_inertial_ x="${panel_thickness}" y="${station_width}" z="${socket_size}" mass="5.0">
       <origin xyz="0 0 0" rpy="0 0 0" />
     </xacro:box_inertial_>
@@ -43,5 +43,5 @@
       <orign rpy="0.0 0.0 0.0" xyz="0.0 0.0 0.0" />
       <geometry>
-        <box size="${panel_thickness} ${pillar_width} ${socket_size}" />
+        <box size="${panel_thickness} ${station_width} ${socket_size}" />
       </geometry>
     </visual>
@@ -49,5 +49,5 @@
       <orign rpy="0.0 0.0 0.0" xyz="0.0 0.0 0.0" />
       <geometry>
-        <box size="${panel_thickness} ${pillar_width} ${socket_size}" />
+        <box size="${panel_thickness} ${station_width} ${socket_size}" />
       </geometry>
     </collision>
@@ -56,8 +56,8 @@
     <parent link="low_body_link" />
     <child link="right_panel_link" />
-    <origin rpy="0.0 0.0 0.0" xyz="${0.25*(pillar_width+socket_size)} 0.0 ${0.5*socket_height + 0.25*socket_size}" />
+    <origin rpy="0.0 0.0 0.0" xyz="${0.25*(station_width+socket_size)} 0.0 ${0.5*socket_height + 0.25*socket_size}" />
   </joint>
   <link name="right_panel_link">
-    <xacro:box_inertial_ x="${panel_thickness}" y="${pillar_width}" z="${socket_size}" mass="5.0">
+    <xacro:box_inertial_ x="${panel_thickness}" y="${station_width}" z="${socket_size}" mass="5.0">
       <origin xyz="0 0 0" rpy="0 0 0" />
     </xacro:box_inertial_>
@@ -65,5 +65,5 @@
       <orign rpy="0.0 0.0 0.0" xyz="0.0 0.0 0.0" />
       <geometry>
-        <box size="${panel_thickness} ${pillar_width} ${socket_size}" />
+        <box size="${panel_thickness} ${station_width} ${socket_size}" />
       </geometry>
     </visual>
@@ -71,5 +71,5 @@
       <orign rpy="0.0 0.0 0.0" xyz="0.0 0.0 0.0" />
       <geometry>
-        <box size="${panel_thickness} ${pillar_width} ${socket_size}" />
+        <box size="${panel_thickness} ${station_width} ${socket_size}" />
       </geometry>
     </collision>
@@ -78,8 +78,8 @@
     <parent link="low_body_link"/>
     <child link="top_panel_link"/>
-    <origin rpy="0.0 0.0 0.0" xyz="0.0 0.0 ${0.25*(2*socket_height + 2*socket_size + pillar_width)}"/>
+    <origin rpy="0.0 0.0 0.0" xyz="0.0 0.0 ${0.25*(2*socket_height + 2*socket_size + station_width)}"/>
   </joint>
   <link name="top_panel_link">
-    <xacro:box_inertial_ x="${pillar_width}" y="${pillar_width}" z="${panel_thickness}" mass="10.0">
+    <xacro:box_inertial_ x="${station_width}" y="${station_width}" z="${panel_thickness}" mass="10.0">
       <origin xyz="0 0 0" rpy="0 0 0" />
     </xacro:box_inertial_>
@@ -87,5 +87,5 @@
       <orign rpy="0.0 0.0 0.0" xyz="0.0 0.0 0.0" />
       <geometry>
-        <box size="${pillar_width} ${pillar_width} ${panel_thickness}" />
+        <box size="${station_width} ${station_width} ${panel_thickness}" />
       </geometry>
     </visual>
@@ -93,9 +93,9 @@
       <orign rpy="0.0 0.0 0.0" xyz="0.0 0.0 0.0" />
       <geometry>
-        <box size="${pillar_width} ${pillar_width} ${panel_thickness}" />
+        <box size="${station_width} ${station_width} ${panel_thickness}" />
       </geometry>
     </collision>
   </link>
-  <!-- colorize pillar -->
+  <!-- colorize adapter station -->
   <gazebo reference="low_body_link">
     <material>Gazebo/Grey</material>
