Commit message: Generate urdf files.

File: _bullet_urdf_autogen/primitive_adapter_station.urdf (robot description, URDF)
Before this commit: robot primitive_adapter_station, 5 links, 4 joints
Links:
- added link target_reference_frame
- added link virt_tgt_frame_x
- added link virt_tgt_frame_y
- added link virt_tgt_frame_z
Joints:
- added joint target_ref_frame_joint: type fixed, parent world, child target_reference_frame, origin xyz=0 -0.125 1.2 rpy=1.5707963267948966 0 3.141592653589793, axis 0 0 0
- added joint virt_tgt_frame_x_joint: type fixed, parent target_reference_frame, child virt_tgt_frame_x, origin xyz=1 0 0 rpy=0 0 0, axis 0 0 0
- added joint virt_tgt_frame_y_joint: type fixed, parent target_reference_frame, child virt_tgt_frame_y, origin xyz=0 1 0 rpy=0 0 0, axis 0 0 0
- added joint virt_tgt_frame_z_joint: type fixed, parent target_reference_frame, child virt_tgt_frame_z, origin xyz=0 0 1 rpy=0 0 0, axis 0 0 0

File: _bullet_urdf_autogen/primitive_chargepal_with_fix_plug.urdf (robot description, URDF)
Before this commit: robot primitive_chargepal_with_gripper, 21 links, 20 joints
Links:
- added link virt_tool_frame_x
- added link virt_tool_frame_y
- added link virt_tool_frame_z
Joints:
- added joint virt_tool_frame_x_joint: type fixed, parent plug_reference_frame, child virt_tool_frame_x, origin xyz=1 0 0 rpy=0 0 0, axis 0 0 0
- added joint virt_tool_frame_y_joint: type fixed, parent plug_reference_frame, child virt_tool_frame_y, origin xyz=0 1 0 rpy=0 0 0, axis 0 0 0
- added joint virt_tool_frame_z_joint: type fixed, parent plug_reference_frame, child virt_tool_frame_z, origin xyz=0 0 1 rpy=0 0 0, axis 0 0 0

Commit message: Add zero mass for virtual links.

File: _bullet_urdf_autogen/primitive_adapter_station.urdf (robot description, URDF)
Before this commit: robot primitive_adapter_station, 9 links, 8 joints
Links:
- link target_reference_frame: mass None -> 0.0
- link virt_tgt_frame_x: mass None -> 0.0
- link virt_tgt_frame_y: mass None -> 0.0
- link virt_tgt_frame_z: mass None -> 0.0

File: _bullet_urdf_autogen/primitive_chargepal_with_fix_plug.urdf (robot description, URDF)
Before this commit: robot primitive_chargepal_with_fix_plug, 24 links, 23 joints
Links:
- link fts_toolside: mass None -> 0.0
- link plug_reference_frame: mass None -> 0.0
- link robotiq_force_torque_frame_id: mass None -> 0.0
- link virt_tool_frame_x: mass None -> 0.0
- link virt_tool_frame_y: mass None -> 0.0
- link virt_tool_frame_z: mass None -> 0.0
- link world: mass None -> 0.0

File: _bullet_urdf_autogen/primitive_chargepal_with_gripper.urdf (robot description, URDF)
Before this commit: robot primitive_chargepal_with_gripper, 31 links, 30 joints
Links:
- link fts_toolside: mass None -> 0.0
- link robotiq_force_torque_frame_id: mass None -> 0.0
- link world: mass None -> 0.0

File: urdf/robotiq_ft_300/robotiq_ft_300.urdf.xacro (robot description, xacro)
@@ -1,4 +1,6 @@
 <?xml version="1.0"?>
 <robot xmlns:xacro="http://ros.org/wiki/xacro" name="robotiq_ft_300">
+  <!-- Macros -->
+  <xacro:include filename="$(find chargepal_description)/urdf/utils/chargepal_common.urdf.xacro" />
   <xacro:macro name="robotiq_ft_300" params="parent prefix *origin">
     <!-- mount the fts to the robot -->
@@ -39,5 +41,6 @@
       <child link="${prefix}robotiq_force_torque_frame_id" />
     </joint>
-    <link name="${prefix}robotiq_force_torque_frame_id"/>
+    <!-- <link name="${prefix}robotiq_force_torque_frame_id"/> -->
+    <xacro:chargepal_virtual_link link_name="${prefix}robotiq_force_torque_frame_id" />
     <!-- toolside frame -->
     <joint name="${prefix}toolside_joint" type="fixed" >
@@ -46,5 +49,6 @@
       <child link="${prefix}fts_toolside" />
     </joint>
-    <link name="${prefix}fts_toolside"/>
+    <!-- <link name="${prefix}fts_toolside"/> -->
+    <xacro:chargepal_virtual_link link_name="${prefix}fts_toolside" />
   </xacro:macro>
 </robot>

File: urdf/utils/chargepal_common.urdf.xacro (robot description, xacro)
@@ -5,5 +5,11 @@
   <!--                                               -->
   <xacro:macro name="chargepal_virtual_link" params="link_name">
-    <link name="${link_name}"/>
+    <link name="${link_name}">
+      <inertial>
+        <mass value="0.0"/>
+        <origin rpy="0 0 0" xyz="0 0 0"/>
+        <inertia ixx="0.0" ixy="0.0" ixz="0.0" iyy="0.0" iyz="0.0" izz="0.0"/>
+      </inertial>
+    </link>
   </xacro:macro>
   <xacro:macro name="chargepal_virtual_joint" params="joint_name type parent child joint_axis_xyz joint_origin_xyz joint_origin_rpy joint_lower_limit joint_upper_limit">

Commit message: Feature: Add inertial properties to the robot links if needed.

File: _bullet_urdf_autogen/primitive_adapter_station.urdf (robot description, URDF)
Before this commit: robot primitive_adapter_station, 9 links, 8 joints
Links:
- link world: mass None -> 0.0

File: _bullet_urdf_autogen/primitive_chargepal_with_fix_plug.urdf (robot description, URDF)
Before this commit: robot primitive_chargepal_with_fix_plug, 24 links, 23 joints
Links:
- link base: mass None -> 0.0
- link base_link: mass None -> 0.0
- link flange: mass None -> 0.0
- link tool0: mass None -> 0.0

File: _bullet_urdf_autogen/primitive_chargepal_with_gripper.urdf (robot description, URDF)
Before this commit: robot primitive_chargepal_with_gripper, 31 links, 30 joints
Links:
- link base: mass None -> 0.0
- link base_link: mass None -> 0.0
- link flange: mass None -> 0.0
- link gripper_tcp: mass None -> 0.0
- link tool0: mass None -> 0.0
