Commit message: Add new tool (plug) and two kind of sockets

File: _bullet_urdf_autogen/primitive_chargepal_with_fix_rod.urdf (robot description, URDF)
Before this commit: robot primitive_chargepal_with_fix_plug, 24 links, 23 joints
Links:
- removed link plug
- removed link plug_border
- added link rod, mass 0.2; collision mesh filename=package://chargepal_tools/plugs/meshes/collision/rod.obj scale=0.001 0.001 0.001; visual mesh filename=package://chargepal_tools/plugs/meshes/visual/rod.obj scale=0.001 0.001 0.001
Joints:
- removed joint plug_border_joint
- removed joint plug_joint
- added joint rod_joint: type fixed, parent fts_toolside, child rod, origin xyz=0.0 0.0 0.035 rpy=0.0 0.0 0.0
- joint plug_ref_frame_joint: origin xyz=0 0 0.015 rpy=0 0 0 -> xyz=0 0 -0.015000000000000003 rpy=0 0 0; parent plug_border -> rod

File: urdf/tools/primitive_fix_plug.urdf.xacro (robot description, xacro)
@@ -11,5 +11,6 @@
   <xacro:property name="length_border" value="0.03" />
   <xacro:property name="mass_plug" value="0.25" />
-  <xacro:property name="radius_plug" value="0.0345" />
+  <xacro:property name="radius_plug" value="0.034" />
+  <!-- <xacro:property name="radius_plug" value="0.0345" /> -->
   <xacro:property name="length_plug" value="0.08" />
   <xacro:macro name="fix_plug" params="parent prefix">

File: urdf/utils/chargepal_material.urdf.xacro (robot description, xacro)
@@ -11,4 +11,9 @@
     <material name="yellow">
       <color rgba="${255/255} ${226/255} ${0/255} 1"/>
+    </material>
+  </xacro:property>
+  <xacro:property name="material_field_green">
+    <material name="field_green">
+      <color rgba="${94/255} ${190/255} ${125/255} 1"/>
     </material>
   </xacro:property>
