Commit message: Add a new chargepal robot with a fix plug as an end-effector.

File: _bullet_urdf_autogen/primitive_chargepal_with_fix_plug.urdf (robot description, URDF)
Before this commit: robot primitive_chargepal_with_gripper, 31 links, 30 joints
Links:
- removed link gripper_coupling_link
- removed link gripper_left_inner_finger
- removed link gripper_left_inner_knuckle
- removed link gripper_left_outer_finger
- removed link gripper_left_outer_knuckle
- removed link gripper_left_robotiq_fingertip_65mm
- removed link gripper_right_inner_finger
- removed link gripper_right_inner_knuckle
- removed link gripper_right_outer_finger
- removed link gripper_right_outer_knuckle
- removed link gripper_right_robotiq_fingertip_65mm
- removed link gripper_robotiq_arg2f_base_link
- removed link gripper_tcp
- added link plug, mass 0.25; collision cylinder length=0.08 radius=0.0345; visual cylinder length=0.08 radius=0.0345
- added link plug_border, mass 0.1; collision cylinder length=0.03 radius=0.045; visual cylinder length=0.03 radius=0.045
- added link plug_reference_frame
Joints:
- removed joint coupling_2f140_joint
- removed joint ft300_coupling_joint
- removed joint gripper_finger_joint
- removed joint gripper_left_fingertip_joint
- removed joint gripper_left_inner_finger_joint
- removed joint gripper_left_inner_knuckle_joint
- removed joint gripper_left_outer_finger_joint
- removed joint gripper_right_fingertip_joint
- removed joint gripper_right_inner_finger_joint
- removed joint gripper_right_inner_knuckle_joint
- removed joint gripper_right_outer_finger_joint
- removed joint gripper_right_outer_knuckle_joint
- removed joint gripper_tcp_joint
- added joint plug_border_joint: type fixed, parent fts_toolside, child plug_border, origin xyz=0.0 0.0 0.015 rpy=0.0 0.0 0.0
- added joint plug_joint: type fixed, parent plug_border, child plug, origin xyz=0.0 0.0 0.055 rpy=0.0 0.0 0.0
- added joint plug_ref_frame_joint: type fixed, parent plug_border, child plug_reference_frame, origin xyz=0 0 0.015 rpy=0 0 0, axis 0 0 0

Commit message: Replacing the force torque sensor with the project specific one

File: _bullet_urdf_autogen/primitive_chargepal_with_fix_plug.urdf (robot description, URDF)
Before this commit: robot primitive_chargepal_with_fix_plug, 24 links, 23 joints
Links:
- removed link fts_robotside
- removed link fts_toolside
- removed link robotiq_force_torque_frame_id
- added link ft_sensor_imu, mass 0.00841533584597687
- added link ft_sensor_mech1, mass 0.0
- added link ft_sensor_mech2, mass 0.0
- added link ft_sensor_mech3, mass 0.0
- added link ft_sensor_mounting, mass 0.14931; collision cylinder length=0.01 radius=0.0315; collision cylinder length=0.028 radius=0.035
- added link ft_sensor_wrench, mass 0.081117
Joints:
- removed joint fts_fix
- removed joint measurement_joint
- removed joint toolside_joint
- added joint mounting_to_imu: type fixed, parent ft_sensor_mounting, child ft_sensor_imu, origin xyz=0 0 0.0093 rpy=0 0 0, axis 0 0 0
- added joint mounting_to_mech1: type fixed, parent ft_sensor_mounting, child ft_sensor_mech1, origin xyz=-0.032879 0 0.0105 rpy=1.5625 0 -1.5708, axis 0 0 0
- added joint mounting_to_mech2: type fixed, parent ft_sensor_mounting, child ft_sensor_mech2, origin xyz=0 -0.032879 0.0105 rpy=1.5708 0 0, axis 0 0 0
- added joint mounting_to_mech3: type fixed, parent ft_sensor_mounting, child ft_sensor_mech3, origin xyz=0.032879 0 0.0105 rpy=1.5708 0 1.5708, axis 0 0 0
- added joint mounting_to_wrench: type fixed, parent ft_sensor_mounting, child ft_sensor_wrench, origin xyz=0 0 0.035 rpy=0 0 0, axis 0 0 0
- added joint ur_to_sensor: type fixed, parent tool0, child ft_sensor_mounting, origin xyz=0.0 0.0 0.0 rpy=0.0 0.0 0.0
- joint plug_border_joint: parent fts_toolside -> ft_sensor_wrench

File: _bullet_urdf_autogen/primitive_chargepal_with_fix_rod.urdf (robot description, URDF)
Before this commit: robot primitive_chargepal_with_fix_rod, 23 links, 22 joints
Links:
- removed link fts_robotside
- removed link fts_toolside
- removed link robotiq_force_torque_frame_id
- added link ft_sensor_imu, mass 0.00841533584597687
- added link ft_sensor_mech1, mass 0.0
- added link ft_sensor_mech2, mass 0.0
- added link ft_sensor_mech3, mass 0.0
- added link ft_sensor_mounting, mass 0.14931; collision cylinder length=0.01 radius=0.0315; collision cylinder length=0.028 radius=0.035
- added link ft_sensor_wrench, mass 0.081117
Joints:
- removed joint fts_fix
- removed joint measurement_joint
- removed joint toolside_joint
- added joint mounting_to_imu: type fixed, parent ft_sensor_mounting, child ft_sensor_imu, origin xyz=0 0 0.0093 rpy=0 0 0, axis 0 0 0
- added joint mounting_to_mech1: type fixed, parent ft_sensor_mounting, child ft_sensor_mech1, origin xyz=-0.032879 0 0.0105 rpy=1.5625 0 -1.5708, axis 0 0 0
- added joint mounting_to_mech2: type fixed, parent ft_sensor_mounting, child ft_sensor_mech2, origin xyz=0 -0.032879 0.0105 rpy=1.5708 0 0, axis 0 0 0
- added joint mounting_to_mech3: type fixed, parent ft_sensor_mounting, child ft_sensor_mech3, origin xyz=0.032879 0 0.0105 rpy=1.5708 0 1.5708, axis 0 0 0
- added joint mounting_to_wrench: type fixed, parent ft_sensor_mounting, child ft_sensor_wrench, origin xyz=0 0 0.035 rpy=0 0 0, axis 0 0 0
- added joint ur_to_sensor: type fixed, parent tool0, child ft_sensor_mounting, origin xyz=0.0 0.0 0.0 rpy=0.0 0.0 0.0
- joint rod_joint: parent fts_toolside -> ft_sensor_wrench

File: _bullet_urdf_autogen/primitive_chargepal_with_gripper.urdf (robot description, URDF)
Before this commit: robot primitive_chargepal_with_gripper, 31 links, 30 joints
Links:
- removed link fts_robotside
- removed link fts_toolside
- removed link robotiq_force_torque_frame_id
- added link ft_sensor_imu, mass 0.00841533584597687
- added link ft_sensor_mech1, mass 0.0
- added link ft_sensor_mech2, mass 0.0
- added link ft_sensor_mech3, mass 0.0
- added link ft_sensor_mounting, mass 0.14931; collision cylinder length=0.01 radius=0.0315; collision cylinder length=0.028 radius=0.035
- added link ft_sensor_wrench, mass 0.081117
Joints:
- removed joint fts_fix
- removed joint measurement_joint
- removed joint toolside_joint
- added joint mounting_to_imu: type fixed, parent ft_sensor_mounting, child ft_sensor_imu, origin xyz=0 0 0.0093 rpy=0 0 0, axis 0 0 0
- added joint mounting_to_mech1: type fixed, parent ft_sensor_mounting, child ft_sensor_mech1, origin xyz=-0.032879 0 0.0105 rpy=1.5625 0 -1.5708, axis 0 0 0
- added joint mounting_to_mech2: type fixed, parent ft_sensor_mounting, child ft_sensor_mech2, origin xyz=0 -0.032879 0.0105 rpy=1.5708 0 0, axis 0 0 0
- added joint mounting_to_mech3: type fixed, parent ft_sensor_mounting, child ft_sensor_mech3, origin xyz=0.032879 0 0.0105 rpy=1.5708 0 1.5708, axis 0 0 0
- added joint mounting_to_wrench: type fixed, parent ft_sensor_mounting, child ft_sensor_wrench, origin xyz=0 0 0.035 rpy=0 0 0, axis 0 0 0
- added joint ur_to_sensor: type fixed, parent tool0, child ft_sensor_mounting, origin xyz=0.0 0.0 0.0 rpy=0.0 0.0 0.0
- joint ft300_coupling_joint: origin xyz=0 0 0.004 rpy=0 0 -1.5707963267948966 -> xyz=0 0 0.007 rpy=0 0 -1.5707963267948966; parent fts_toolside -> ft_sensor_wrench

File: urdf/bringups/primitive_chargepal_with_fix_plug.urdf.xacro (robot description, xacro)
@@ -67,12 +67,15 @@
     <selfCollide>true</selfCollide>
   </gazebo>
-  <!-- ############## FT SENSOR ############### -->
-  <xacro:include filename="$(find chargepal_description)/urdf/robotiq_ft_300/robotiq_ft_300.urdf.xacro" />
-  <xacro:robotiq_ft_300 parent="${prefix}tool0" prefix="${prefix}">
-    <origin xyz="0 0 0" rpy="0 0 0" />
-  </xacro:robotiq_ft_300>
+  <!-- ############### Bota Systems SensONE FT SENSOR-->
+  <xacro:include filename="$(find rokubimini_description)/urdf/BFT_SENS_ECAT_M8.urdf.xacro" />
+  <xacro:BFT_SENS_ECAT_M8 prefix="${prefix}ft_sensor" />
+  <joint name="ur_to_sensor" type="fixed">
+    <parent link="${prefix}tool0" />
+    <child link="${prefix}ft_sensor_mounting" />
+    <origin xyz="0.0 0.0 0.0" rpy="0.0 0.0 0.0" />
+  </joint>
   <!-- ############### FIX PLUG ################ -->
   <xacro:include filename="$(find chargepal_description)/urdf/tools/primitive_fix_plug.urdf.xacro" />
-  <xacro:fix_plug parent="${prefix}fts_toolside" prefix="${prefix}" />
+  <xacro:fix_plug parent="${prefix}ft_sensor_wrench" prefix="${prefix}" />
   <!-- Add three (for each axis) additional virtual frames for reward calculation -->
   <xacro:chargepal_virtual_joint

File: urdf/bringups/primitive_chargepal_with_fix_rod.urdf.xacro (robot description, xacro)
@@ -67,12 +67,15 @@
     <selfCollide>true</selfCollide>
   </gazebo>
-  <!-- ############## FT SENSOR ############### -->
-  <xacro:include filename="$(find chargepal_description)/urdf/robotiq_ft_300/robotiq_ft_300.urdf.xacro" />
-  <xacro:robotiq_ft_300 parent="${prefix}tool0" prefix="${prefix}">
-    <origin xyz="0 0 0" rpy="0 0 0" />
-  </xacro:robotiq_ft_300>
+  <!-- ############### Bota Systems SensONE FT SENSOR-->
+  <xacro:include filename="$(find rokubimini_description)/urdf/BFT_SENS_ECAT_M8.urdf.xacro" />
+  <xacro:BFT_SENS_ECAT_M8 prefix="${prefix}ft_sensor" />
+  <joint name="ur_to_sensor" type="fixed">
+    <parent link="${prefix}tool0" />
+    <child link="${prefix}ft_sensor_mounting" />
+    <origin xyz="0.0 0.0 0.0" rpy="0.0 0.0 0.0" />
+  </joint>
   <!-- ############### FIX PLUG ################ -->
   <xacro:include filename="$(find chargepal_tools)/urdf/rod.urdf.xacro" />
-  <xacro:rod_tool parent="${prefix}fts_toolside" prefix="${prefix}" />
+  <xacro:rod_tool parent="${prefix}ft_sensor_wrench" prefix="${prefix}" />
   <!-- Add three (for each axis) additional virtual frames for reward calculation -->
   <xacro:chargepal_virtual_joint

File: urdf/bringups/primitive_chargepal_with_gripper.urdf.xacro (robot description, xacro)
@@ -65,9 +65,12 @@
     <selfCollide>true</selfCollide>
   </gazebo>
-  <!-- ############## FT SENSOR ############### -->
-  <xacro:include filename="$(find chargepal_description)/urdf/robotiq_ft_300/robotiq_ft_300.urdf.xacro" />
-  <xacro:robotiq_ft_300 parent="${prefix}tool0" prefix="${prefix}">
-    <origin xyz="0 0 0" rpy="0 0 0" />
-  </xacro:robotiq_ft_300>
+  <!-- ############### Bota Systems SensONE FT SENSOR-->
+  <xacro:include filename="$(find rokubimini_description)/urdf/BFT_SENS_ECAT_M8.urdf.xacro" />
+  <xacro:BFT_SENS_ECAT_M8 prefix="${prefix}ft_sensor" />
+  <joint name="ur_to_sensor" type="fixed">
+    <parent link="${prefix}tool0" />
+    <child link="${prefix}ft_sensor_mounting" />
+    <origin xyz="0.0 0.0 0.0" rpy="0.0 0.0 0.0" />
+  </joint>
   <!-- ############### GRIPPER ################ -->
   <xacro:include filename="$(find chargepal_description)/urdf/robotiq_2f_140/robotiq_arg2f_140_model_macro.xacro" />
@@ -78,6 +81,6 @@
   <xacro:property name="coupling_mass" value="0.100" />
   <joint name="${prefix}ft300_coupling_joint" type="fixed">
-    <origin xyz="0 0 ${coupling_inner_length / 2}" rpy="0 0 ${-pi/2}" />
-    <parent link="${prefix}fts_toolside" />
+    <origin xyz="0 0 ${coupling_outer_length / 2}" rpy="0 0 ${-pi/2}" />
+    <parent link="${prefix}ft_sensor_wrench" />
     <child link="${prefix}gripper_coupling_link" />
   </joint>

File: urdf/robotiq_ft_300/robotiq_ft_300.urdf.xacro (robot description, xacro)
@@ -45,6 +45,6 @@
     <!-- toolside frame -->
     <joint name="${prefix}toolside_joint" type="fixed" >
-      <origin xyz="0 0 0.0375" rpy="0 0 0" />
-      <parent link="${prefix}fts_robotside" />
+      <origin xyz="0 0 0.02125" rpy="0 0 0" />
+      <parent link="${prefix}robotiq_force_torque_frame_id" />
       <child link="${prefix}fts_toolside" />
     </joint>
