Commit message: Add pink as new material

File: urdf/utils/chargepal_material.urdf.xacro (robot description, xacro)
@@ -11,4 +11,9 @@
     <material name="yellow">
       <color rgba="${255/255} ${226/255} ${0/255} 1"/>
+    </material>
+  </xacro:property>
+  <xacro:property name="material_pink">
+    <material name="pink">
+      <color rgba="0.937 0.109 0.882 1"/>
     </material>
   </xacro:property>

File: urdf/utils/common_properties.urdf.xacro (robot description, xacro)
@@ -1,4 +1,5 @@
 <?xml version="1.0" ?>
 <!-- Various useful properties such as constants and materials -->
+<!-- TODO: change include paths in xacro files to chargepal_inertial and chargpal_material -->
 <robot name="xacro_properties" xmlns:xacro="http://ros.org/wiki/xacro">
   <!-- #################### RViz materials #################### -->

Commit message: Add testbed description

File: urdf/utils/chargepal_material.urdf.xacro (robot description, xacro)
@@ -48,4 +48,14 @@
     </material>
   </xacro:property>
+  <xacro:property name="material_vention_green">
+    <material name="vention_green">
+      <color rgba="${12/255} ${129/255} ${138/255} 1"/>
+    </material>
+  </xacro:property>
+  <xacro:property name="material_vention_blue">
+    <material name="vention_blue">
+      <color rgba="${32/255} ${120/255} ${170/255} 1"/>
+    </material>
+  </xacro:property>
   <xacro:property name="material_aluminium">
     <material name="aluminium">
