Commit message: Update of the arm joint limits back to the original values

File: _bullet_urdf_models/chargepal_testbed_fix_rod.urdf (robot description, URDF)
Before this commit: robot chargepal_testbed, 26 links, 25 joints
Joints:
- joint elbow_joint: limit lower=-3.141592653589793 upper=0.0 effort=150.0 velocity=3.141592653589793 -> lower=-3.141592653589793 upper=3.141592653589793 effort=150.0 velocity=3.141592653589793
- joint shoulder_lift_joint: limit lower=-3.141592653589793 upper=0.0 effort=330.0 velocity=3.141592653589793 -> lower=-6.283185307179586 upper=6.283185307179586 effort=330.0 velocity=2.0943951023931953
- joint shoulder_pan_joint: limit lower=-3.141592653589793 upper=3.141592653589793 effort=330.0 velocity=3.141592653589793 -> lower=-6.283185307179586 upper=6.283185307179586 effort=330.0 velocity=2.0943951023931953
- joint testbed_to_ur10e: origin xyz=0.0 0.0 0.0 rpy=0.0 0.0 1.570795 -> xyz=0.0 0.0 0.0 rpy=0.0 0.0 -1.570795
- joint wrist_1_joint: limit lower=-3.141592653589793 upper=3.141592653589793 effort=56.0 velocity=3.141592653589793 -> lower=-6.283185307179586 upper=6.283185307179586 effort=56.0 velocity=3.141592653589793
- joint wrist_2_joint: limit lower=-3.141592653589793 upper=3.141592653589793 effort=56.0 velocity=3.141592653589793 -> lower=-6.283185307179586 upper=6.283185307179586 effort=56.0 velocity=3.141592653589793
- joint wrist_3_joint: limit lower=-0.7853981633974483 upper=5.497787143782138 effort=56.0 velocity=3.141592653589793 -> lower=-6.283185307179586 upper=6.283185307179586 effort=56.0 velocity=3.141592653589793

File: urdf/bringups/chargepal_testbed_fix_rod.urdf.xacro (robot description, xacro)
@@ -13,10 +13,10 @@
     <parent link="${prefix}arm_base" />
     <child link="${prefix}base_link" />
-    <origin xyz="0.0 0.0 0.0" rpy="0.0 0.0 ${0.5*M_PI}" />
+    <origin xyz="0.0 0.0 0.0" rpy="0.0 0.0 ${-0.5*M_PI}" />
   </joint>
   <!-- ############### UR10e ARM ################ -->
   <xacro:include filename="$(find ur_description)/urdf/inc/ur10e_macro.xacro"/>
   <!-- Arguments to load UR10e arm macro -->
-  <xacro:arg name="joint_limit_params" default="$(find chargepal_description)/config/ur10e/joint_limits.yaml"/>
+  <xacro:arg name="joint_limit_params" default="$(find ur_description)/config/ur10e/joint_limits.yaml"/>
   <xacro:arg name="physical_params" default="$(find ur_description)/config/ur10e/physical_parameters.yaml"/>
   <xacro:arg name="kinematics_params" default="$(find ur_description)/config/ur10e/default_kinematics.yaml"/>

Commit message: Add testbed description with top-down task

File: _bullet_urdf_models/chargepal_testbed_fix_rod.urdf (robot description, URDF)
Before this commit: robot chargepal_testbed, 26 links, 25 joints
Links:
- link table: geometry collision box size=0.81 1.215 0.8136; visual mesh filename=package://chargepal_description/meshes/testbed/table.dae
Joints:
- joint baseplate_to_arm: origin xyz=0 0 0.01125 rpy=0 0 0 -> xyz=0 0 0.0225 rpy=0 0 0
- joint table_to_baseplate: origin xyz=0.45 -0.24750000000000005 0.418035 rpy=0 0 -1.570795 -> xyz=-0.1575 -0.1575 0 rpy=0 0 3.14159
- joint world_to_table: origin xyz=0 0 0.406785 rpy=0 0 1.570795 -> xyz=0 0 0 rpy=0 0 3.14159

File: _bullet_urdf_models/testbed_table.urdf (robot description, URDF)
Before this commit: robot testbed, 4 links, 3 joints
Links:
- link table: geometry collision box size=0.81 1.215 0.8136; visual mesh filename=package://chargepal_description/meshes/testbed/table.dae
Joints:
- joint baseplate_to_arm: origin xyz=0 0 0.01125 rpy=0 0 0 -> xyz=0 0 0.0225 rpy=0 0 0
- joint table_to_baseplate: origin xyz=0.45 -0.24750000000000005 0.418035 rpy=0 0 -1.570795 -> xyz=-0.1575 -0.1575 0 rpy=0 0 3.14159
- joint world_to_table: origin xyz=0 0 0.406785 rpy=0 0 1.570795 -> xyz=0 0 0 rpy=0 0 3.14159

File: urdf/environment/testbed_table.urdf.xacro (robot description, xacro)
@@ -11,6 +11,7 @@
   <xacro:property name="M_PI" value="3.14159"/>
   <!-- object properties -->
-  <xacro:property name="table_length" value="1.215" />
-  <xacro:property name="table_width" value="0.81" />
+  <xacro:property name="table_width" value="1.215" />
+  <xacro:property name="table_length" value="0.81" />
+  <xacro:property name="table_height" value="0.8136" />
   <xacro:property name="table_mesh_length" value="1.249" />
   <xacro:property name="table_mesh_width" value="0.84398" />
@@ -24,21 +25,21 @@
     <parent link="world"/>
     <child link="${prefix}table"/>
-    <origin xyz="0 0 ${table_mesh_height/2}" rpy="0 0 ${M_PI/2}"/>
+    <origin xyz="0 0 0" rpy="0 0 ${M_PI}"/>
   </joint>
   <link name="${prefix}table">
-    <xacro:inertial_box x="${table_mesh_length}" y="${table_mesh_width}" z="${table_mesh_height}" mass="100.0">
+    <xacro:inertial_box x="${table_length}" y="${table_width}" z="${table_height}" mass="100.0">
       <origin xyz="0 0 0" rpy="0 0 0" />
     </xacro:inertial_box>
     <visual>
-      <origin xyz="${-table_mesh_length/2-0.006} ${-table_mesh_width/2-0.011} ${-table_mesh_height/2-0.0052}" rpy="${M_PI/2} 0.0 ${M_PI/2}" />
+      <origin xyz="0 0 0" rpy="0 0 0" />
       <geometry>
-        <mesh filename="package://chargepal_description/meshes/testbed/table.stl" />
+        <mesh filename="package://chargepal_description/meshes/testbed/table.dae" />
       </geometry>
       <xacro:insert_block name="material_vention_green" />
     </visual>
     <collision>
-      <origin xyz="0.0 0.0 0.0" rpy="0.0 0.0 0.0" />
+      <origin xyz="${-table_length/2} ${-table_width/2} ${-table_height/2}" rpy="0.0 0.0 0.0" />
       <geometry>
-        <box size="${table_mesh_length} ${table_mesh_width} ${table_mesh_height}" />
+        <box size="${table_length} ${table_width} ${table_height}" />
       </geometry>
     </collision>
@@ -48,6 +49,6 @@
     <child link="${prefix}base_plate"/>
     <origin
-      xyz="${table_length/2 - profile_size - baseplate_size/2} ${-table_width/2 + profile_size + baseplate_size/2} ${table_mesh_height/2 + baseplate_height/2}"
-      rpy="0 0 ${-M_PI/2}"/>
+      xyz="${-profile_size - baseplate_size/2} ${-profile_size - baseplate_size/2} 0"
+      rpy="0 0 ${M_PI}"/>
   </joint>
   <link name="${prefix}base_plate">
@@ -56,12 +57,12 @@
     </xacro:inertial_box>
     <visual>
-      <origin xyz="${-baseplate_size/2} ${-baseplate_size/2} ${-baseplate_height/2}" rpy="${M_PI/2} 0.0 ${M_PI/2}" />
+      <origin xyz="0 0 0" rpy="0 0 0" />
       <geometry>
-        <mesh filename="package://chargepal_description/meshes/testbed/base_plate_ur10e.stl" />
+        <mesh filename="package://chargepal_description/meshes/testbed/base_plate_ur10e.dae" />
       </geometry>
       <xacro:insert_block name="material_vention_blue" />
     </visual>
     <collision>
-      <origin xyz="0.0 0.0 0.0" rpy="0.0 0.0 0.0" />
+      <origin xyz="0.0 0.0 ${baseplate_height/2}" rpy="0.0 0.0 0.0" />
       <geometry>
         <box size="${baseplate_size} ${baseplate_size} ${baseplate_height}" />
@@ -73,5 +74,5 @@
     <child link="${prefix}arm_base"/>
     <origin
-      xyz="0 0 ${baseplate_height/2}"
+      xyz="0 0 ${baseplate_height}"
       rpy="0 0 0"/>
   </joint>

Commit message: Remove virtual links

File: _bullet_urdf_models/chargepal_testbed_fix_rod.urdf (robot description, URDF)
Before this commit: robot chargepal_testbed, 26 links, 25 joints
Links:
- removed link virt_tool_frame_x
- removed link virt_tool_frame_y
- removed link virt_tool_frame_z
Joints:
- removed joint virt_tool_frame_x_joint
- removed joint virt_tool_frame_y_joint
- removed joint virt_tool_frame_z_joint

File: _bullet_urdf_models/primitive_chargepal_with_fix_plug.urdf (robot description, URDF)
Before this commit: robot primitive_chargepal_with_fix_plug, 27 links, 26 joints
Links:
- removed link virt_tool_frame_x
- removed link virt_tool_frame_y
- removed link virt_tool_frame_z
Joints:
- removed joint virt_tool_frame_x_joint
- removed joint virt_tool_frame_y_joint
- removed joint virt_tool_frame_z_joint

File: urdf/bringups/chargepal_testbed_fix_rod.urdf.xacro (robot description, xacro)
@@ -79,41 +79,4 @@
   <xacro:include filename="$(find chargepal_tools)/urdf/rod.urdf.xacro" />
   <xacro:rod_tool parent="${prefix}ft_sensor_wrench" prefix="${prefix}" diameter="${ROD_DIAMETER}" />
-  <!-- Add three (for each axis) additional virtual frames for reward calculation -->
-  <xacro:chargepal_virtual_joint
-    joint_name="${prefix}virt_tool_frame_x_joint"
-    type="fixed"
-    parent="${prefix}plug_reference_frame"
-    child="${prefix}virt_tool_frame_x"
-    joint_axis_xyz="0 0 0"
-    joint_origin_xyz="1 0 0"
-    joint_origin_rpy="0 0 0"
-    joint_lower_limit="0"
-    joint_upper_limit="0"
-  />
-  <xacro:chargepal_virtual_link link_name="${prefix}virt_tool_frame_x" />
-  <xacro:chargepal_virtual_joint
-    joint_name="${prefix}virt_tool_frame_y_joint"
-    type="fixed"
-    parent="${prefix}plug_reference_frame"
-    child="${prefix}virt_tool_frame_y"
-    joint_axis_xyz="0 0 0"
-    joint_origin_xyz="0 1 0"
-    joint_origin_rpy="0 0 0"
-    joint_lower_limit="0"
-    joint_upper_limit="0"
-  />
-  <xacro:chargepal_virtual_link link_name="${prefix}virt_tool_frame_y" />
-  <xacro:chargepal_virtual_joint
-    joint_name="${prefix}virt_tool_frame_z_joint"
-    type="fixed"
-    parent="${prefix}plug_reference_frame"
-    child="${prefix}virt_tool_frame_z"
-    joint_axis_xyz="0 0 0"
-    joint_origin_xyz="0 0 1"
-    joint_origin_rpy="0 0 0"
-    joint_lower_limit="0"
-    joint_upper_limit="0"
-  />
-  <xacro:chargepal_virtual_link link_name="${prefix}virt_tool_frame_z" />
   <!-- ################ GAZEBO ################ -->
   <!-- Common -->

File: urdf/bringups/cpm_fix_rod_macro.urdf.xacro (robot description, xacro)
@@ -79,41 +79,4 @@
     <xacro:include filename="$(find chargepal_tools)/urdf/rod.urdf.xacro" />
     <xacro:rod_tool parent="${prefix}ft_sensor_wrench" prefix="${prefix}" diameter="${rod_diameter}" />
-    <!-- Add three (for each axis) additional virtual frames for reward calculation -->
-    <xacro:chargepal_virtual_joint
-        joint_name="${prefix}virt_tool_frame_x_joint"
-        type="fixed"
-        parent="${prefix}plug_reference_frame"
-        child="${prefix}virt_tool_frame_x"
-        joint_axis_xyz="0 0 0"
-        joint_origin_xyz="1 0 0"
-        joint_origin_rpy="0 0 0"
-        joint_lower_limit="0"
-        joint_upper_limit="0"
-    />
-    <xacro:chargepal_virtual_link link_name="${prefix}virt_tool_frame_x" />
-    <xacro:chargepal_virtual_joint
-        joint_name="${prefix}virt_tool_frame_y_joint"
-        type="fixed"
-        parent="${prefix}plug_reference_frame"
-        child="${prefix}virt_tool_frame_y"
-        joint_axis_xyz="0 0 0"
-        joint_origin_xyz="0 1 0"
-        joint_origin_rpy="0 0 0"
-        joint_lower_limit="0"
-        joint_upper_limit="0"
-    />
-    <xacro:chargepal_virtual_link link_name="${prefix}virt_tool_frame_y" />
-    <xacro:chargepal_virtual_joint
-        joint_name="${prefix}virt_tool_frame_z_joint"
-        type="fixed"
-        parent="${prefix}plug_reference_frame"
-        child="${prefix}virt_tool_frame_z"
-        joint_axis_xyz="0 0 0"
-        joint_origin_xyz="0 0 1"
-        joint_origin_rpy="0 0 0"
-        joint_lower_limit="0"
-        joint_upper_limit="0"
-    />
-    <xacro:chargepal_virtual_link link_name="${prefix}virt_tool_frame_z" />
     <!-- ################ GAZEBO ################ -->
     <!-- Common -->

File: urdf/bringups/primitive_chargepal_with_fix_plug.urdf.xacro (robot description, xacro)
@@ -78,41 +78,4 @@
   <xacro:include filename="$(find chargepal_description)/urdf/tools/primitive_fix_plug.urdf.xacro" />
   <xacro:fix_plug parent="${prefix}ft_sensor_wrench" prefix="${prefix}" />
-  <!-- Add three (for each axis) additional virtual frames for reward calculation -->
-  <xacro:chargepal_virtual_joint
-    joint_name="${prefix}virt_tool_frame_x_joint"
-    type="fixed"
-    parent="${prefix}plug_reference_frame"
-    child="${prefix}virt_tool_frame_x"
-    joint_axis_xyz="0 0 0"
-    joint_origin_xyz="1 0 0"
-    joint_origin_rpy="0 0 0"
-    joint_lower_limit="0"
-    joint_upper_limit="0"
-  />
-  <xacro:chargepal_virtual_link link_name="${prefix}virt_tool_frame_x" />
-  <xacro:chargepal_virtual_joint
-    joint_name="${prefix}virt_tool_frame_y_joint"
-    type="fixed"
-    parent="${prefix}plug_reference_frame"
-    child="${prefix}virt_tool_frame_y"
-    joint_axis_xyz="0 0 0"
-    joint_origin_xyz="0 1 0"
-    joint_origin_rpy="0 0 0"
-    joint_lower_limit="0"
-    joint_upper_limit="0"
-  />
-  <xacro:chargepal_virtual_link link_name="${prefix}virt_tool_frame_y" />
-  <xacro:chargepal_virtual_joint
-    joint_name="${prefix}virt_tool_frame_z_joint"
-    type="fixed"
-    parent="${prefix}plug_reference_frame"
-    child="${prefix}virt_tool_frame_z"
-    joint_axis_xyz="0 0 0"
-    joint_origin_xyz="0 0 1"
-    joint_origin_rpy="0 0 0"
-    joint_lower_limit="0"
-    joint_upper_limit="0"
-  />
-  <xacro:chargepal_virtual_link link_name="${prefix}virt_tool_frame_z" />
   <!-- ################ GAZEBO ################ -->
   <!-- Common -->
