Commit message: Name all reference links the same

File: _bullet_urdf_models/adapter_station_octa_socket.urdf (robot description, URDF)
Before this commit: robot adapter_station_square_socket, 7 links, 6 joints
Links:
- removed link socket_link
- removed link target_reference_frame
- removed link virt_tgt_frame_x
- removed link virt_tgt_frame_y
- removed link virt_tgt_frame_z
- added link socket, mass 0.0
- added link station_socket, mass 2.0; collision mesh filename=package://chargepal_tools/sockets/meshes/collision/octagona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 scale=0.001 0.001 0.001; visual mesh filename=package://chargepal_tools/sockets/meshes/visual/octagonal_h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 scale=0.001 0.001 0.001
Joints:
- removed joint target_ref_frame_joint
- removed joint virt_tgt_frame_x_joint
- removed joint virt_tgt_frame_y_joint
- removed joint virt_tgt_frame_z_joint
- added joint station_socket_joint: type fixed, parent world, child station_socket, origin xyz=0.0 0.0 1.2 rpy=1.5707963267948966 0.0 0.0
- joint socket_joint: axis (none) -> 0 0 0; child socket_link -> socket; origin xyz=0.0 0.0 1.2 rpy=1.5707963267948966 0.0 0.0 -> xyz=0 -0.05 1.2 rpy=1.5707963267948966 0 3.141592653589793

File: _bullet_urdf_models/adapter_station_square_socket.urdf (robot description, URDF)
Before this commit: robot adapter_station_square_socket, 7 links, 6 joints
Links:
- removed link socket_link
- removed link target_reference_frame
- removed link virt_tgt_frame_x
- removed link virt_tgt_frame_y
- removed link virt_tgt_frame_z
- added link socket, mass 0.0
- added link station_socket, mass 2.0; collision mesh filename=package://chargepal_tools/sockets/meshes/collision/square_h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 scale=0.001 0.001 0.001; visual mesh filename=package://chargepal_tools/sockets/meshes/visual/square_hole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 scale=0.001 0.001 0.001
Joints:
- removed joint target_ref_frame_joint
- removed joint virt_tgt_frame_x_joint
- removed joint virt_tgt_frame_y_joint
- removed joint virt_tgt_frame_z_joint
- added joint station_socket_joint: type fixed, parent world, child station_socket, origin xyz=0.0 0.0 1.2 rpy=1.5707963267948966 0.0 0.0
- joint socket_joint: axis (none) -> 0 0 0; child socket_link -> socket; origin xyz=0.0 0.0 1.2 rpy=1.5707963267948966 0.0 0.0 -> xyz=0 -0.05 1.2 rpy=1.5707963267948966 0 3.141592653589793

File: _bullet_urdf_models/chargepal_testbed_fix_rod.urdf (robot description, URDF)
Before this commit: robot chargepal_testbed, 23 links, 22 joints
Links:
- removed link plug_reference_frame
- added link plug, mass 0.0
Joints:
- removed joint plug_ref_frame_joint
- added joint plug_joint: type fixed, parent rod, child plug, origin xyz=0 0 -0.015000000000000003 rpy=0 0 0, axis 0 0 0

File: _bullet_urdf_models/chargepal_testbed_tdt.urdf (robot description, URDF)
Before this commit: robot chargepal_testbed, 23 links, 22 joints
Joints:
- removed joint plug_ref_frame_joint
- added joint plug_joint: type fixed, parent plug_root, child plug, origin xyz=0 0 0.02 rpy=0 0 0, axis 0 0 0

File: _bullet_urdf_models/cpm_fix_rod_30.urdf (robot description, URDF)
Before this commit: robot cpm_fix_rod_30, 26 links, 25 joints
Links:
- removed link plug_reference_frame
- removed link virt_tool_frame_x
- removed link virt_tool_frame_y
- removed link virt_tool_frame_z
- added link plug, mass 0.0
Joints:
- removed joint plug_ref_frame_joint
- removed joint virt_tool_frame_x_joint
- removed joint virt_tool_frame_y_joint
- removed joint virt_tool_frame_z_joint
- added joint plug_joint: type fixed, parent rod, child plug, origin xyz=0 0 -0.015000000000000003 rpy=0 0 0, axis 0 0 0

File: _bullet_urdf_models/cpm_fix_rod_32d5.urdf (robot description, URDF)
Before this commit: robot cpm_fix_rod_30, 26 links, 25 joints
Links:
- removed link plug_reference_frame
- removed link virt_tool_frame_x
- removed link virt_tool_frame_y
- removed link virt_tool_frame_z
- added link plug, mass 0.0
Joints:
- removed joint plug_ref_frame_joint
- removed joint virt_tool_frame_x_joint
- removed joint virt_tool_frame_y_joint
- removed joint virt_tool_frame_z_joint
- added joint plug_joint: type fixed, parent rod, child plug, origin xyz=0 0 -0.015000000000000003 rpy=0 0 0, axis 0 0 0

File: _bullet_urdf_models/cpm_fix_rod_34.urdf (robot description, URDF)
Before this commit: robot cpm_fix_rod_30, 26 links, 25 joints
Links:
- removed link plug_reference_frame
- removed link virt_tool_frame_x
- removed link virt_tool_frame_y
- removed link virt_tool_frame_z
- added link plug, mass 0.0
Joints:
- removed joint plug_ref_frame_joint
- removed joint virt_tool_frame_x_joint
- removed joint virt_tool_frame_y_joint
- removed joint virt_tool_frame_z_joint
- added joint plug_joint: type fixed, parent rod, child plug, origin xyz=0 0 -0.015000000000000003 rpy=0 0 0, axis 0 0 0

File: _bullet_urdf_models/cpm_fix_rod_34d5.urdf (robot description, URDF)
Before this commit: robot cpm_fix_rod_30, 26 links, 25 joints
Links:
- removed link plug_reference_frame
- removed link virt_tool_frame_x
- removed link virt_tool_frame_y
- removed link virt_tool_frame_z
- added link plug, mass 0.0
Joints:
- removed joint plug_ref_frame_joint
- removed joint virt_tool_frame_x_joint
- removed joint virt_tool_frame_y_joint
- removed joint virt_tool_frame_z_joint
- added joint plug_joint: type fixed, parent rod, child plug, origin xyz=0 0 -0.015000000000000003 rpy=0 0 0, axis 0 0 0

File: _bullet_urdf_models/fix_rod_30.urdf (robot description, URDF)
Before this commit: robot fix_rod_30, 6 links, 5 joints
Links:
- removed link plug_reference_frame
- removed link virt_tool_frame_x
- removed link virt_tool_frame_y
- removed link virt_tool_frame_z
- added link plug, mass 0.0
Joints:
- removed joint plug_ref_frame_joint
- removed joint virt_tool_frame_x_joint
- removed joint virt_tool_frame_y_joint
- removed joint virt_tool_frame_z_joint
- added joint plug_joint: type fixed, parent rod, child plug, origin xyz=0 0 -0.015000000000000003 rpy=0 0 0, axis 0 0 0

File: _bullet_urdf_models/primitive_adapter_station.urdf (robot description, URDF)
Before this commit: robot primitive_adapter_station, 9 links, 8 joints
Links:
- removed link target_reference_frame
- removed link virt_tgt_frame_x
- removed link virt_tgt_frame_y
- removed link virt_tgt_frame_z
- added link socket, mass 0.0
Joints:
- removed joint target_ref_frame_joint
- removed joint virt_tgt_frame_x_joint
- removed joint virt_tgt_frame_y_joint
- removed joint virt_tgt_frame_z_joint
- added joint socket_joint: type fixed, parent world, child socket, origin xyz=0 -0.125 1.2 rpy=1.5707963267948966 0 3.141592653589793, axis 0 0 0

File: _bullet_urdf_models/primitive_chargepal_with_fix_plug.urdf (robot description, URDF)
Before this commit: robot primitive_chargepal_with_fix_plug, 24 links, 23 joints
Links:
- removed link plug_reference_frame
- added link plug_rod, mass 0.25; collision cylinder length=0.08 radius=0.034; visual cylinder length=0.08 radius=0.034
- link plug: mass 0.25 -> 0.0; geometry 
Joints:
- removed joint plug_ref_frame_joint
- added joint plug_rod_joint: type fixed, parent plug_border, child plug_rod, origin xyz=0.0 0.0 0.055 rpy=0.0 0.0 0.0
- joint plug_joint: axis (none) -> 0 0 0; origin xyz=0.0 0.0 0.055 rpy=0.0 0.0 0.0 -> xyz=0 0 0.015 rpy=0 0 0

File: urdf/environment/primitive_adapter_station.urdf.xacro (robot description, xacro)
@@ -107,8 +107,8 @@
   <!-- virtual target reference frame -->
   <xacro:chargepal_virtual_joint
-    joint_name="target_ref_frame_joint"
+    joint_name="socket_joint"
     type="fixed"
     parent="world"
-    child="target_reference_frame"
+    child="socket"
     joint_axis_xyz="0 0 0"
     joint_origin_xyz="0 ${-station_width/2} ${socket_height}"
@@ -117,42 +117,5 @@
     joint_upper_limit="0"
   />
-  <xacro:chargepal_virtual_link link_name="target_reference_frame" />
-  <!-- Add three (for each axis) additional virtual frames for reward calculation -->
-  <xacro:chargepal_virtual_joint
-    joint_name="virt_tgt_frame_x_joint"
-    type="fixed"
-    parent="target_reference_frame"
-    child="virt_tgt_frame_x"
-    joint_axis_xyz="0 0 0"
-    joint_origin_xyz="1 0 0"
-    joint_origin_rpy="0 0 0"
-    joint_lower_limit="0"
-    joint_upper_limit="0"
-  />
-  <xacro:chargepal_virtual_link link_name="virt_tgt_frame_x" />
-  <xacro:chargepal_virtual_joint
-    joint_name="virt_tgt_frame_y_joint"
-    type="fixed"
-    parent="target_reference_frame"
-    child="virt_tgt_frame_y"
-    joint_axis_xyz="0 0 0"
-    joint_origin_xyz="0 1 0"
-    joint_origin_rpy="0 0 0"
-    joint_lower_limit="0"
-    joint_upper_limit="0"
-  />
-  <xacro:chargepal_virtual_link link_name="virt_tgt_frame_y" />
-  <xacro:chargepal_virtual_joint
-    joint_name="virt_tgt_frame_z_joint"
-    type="fixed"
-    parent="target_reference_frame"
-    child="virt_tgt_frame_z"
-    joint_axis_xyz="0 0 0"
-    joint_origin_xyz="0 0 1"
-    joint_origin_rpy="0 0 0"
-    joint_lower_limit="0"
-    joint_upper_limit="0"
-  />
-  <xacro:chargepal_virtual_link link_name="virt_tgt_frame_z" />
+  <xacro:chargepal_virtual_link link_name="socket" />
   <!-- colorize adapter station -->
   <gazebo reference="low_body_link">

File: urdf/tools/fix_rod_macro.urdf.xacro (robot description, xacro)
@@ -6,41 +6,4 @@
     <link name="world"/>
     <xacro:rod_tool parent="world" prefix="${prefix}" diameter="${rod_diameter}" />
-    <!-- Add three (for each axis) additional virtual frames for reward calculation -->
-    <xacro:chargepal_virtual_joint
-        joint_name="${prefix}virt_tool_frame_x_joint"
-        type="fixed"
-        parent="${prefix}plug_reference_frame"
-        child="${prefix}virt_tool_frame_x"
-        joint_axis_xyz="0 0 0"
-        joint_origin_xyz="1 0 0"
-        joint_origin_rpy="0 0 0"
-        joint_lower_limit="0"
-        joint_upper_limit="0"
-    />
-    <xacro:chargepal_virtual_link link_name="${prefix}virt_tool_frame_x" />
-    <xacro:chargepal_virtual_joint
-        joint_name="${prefix}virt_tool_frame_y_joint"
-        type="fixed"
-        parent="${prefix}plug_reference_frame"
-        child="${prefix}virt_tool_frame_y"
-        joint_axis_xyz="0 0 0"
-        joint_origin_xyz="0 1 0"
-        joint_origin_rpy="0 0 0"
-        joint_lower_limit="0"
-        joint_upper_limit="0"
-    />
-    <xacro:chargepal_virtual_link link_name="${prefix}virt_tool_frame_y" />
-    <xacro:chargepal_virtual_joint
-        joint_name="${prefix}virt_tool_frame_z_joint"
-        type="fixed"
-        parent="${prefix}plug_reference_frame"
-        child="${prefix}virt_tool_frame_z"
-        joint_axis_xyz="0 0 0"
-        joint_origin_xyz="0 0 1"
-        joint_origin_rpy="0 0 0"
-        joint_lower_limit="0"
-        joint_upper_limit="0"
-    />
-    <xacro:chargepal_virtual_link link_name="${prefix}virt_tool_frame_z" />
   </xacro:macro>
 </robot>

File: urdf/tools/primitive_fix_plug.urdf.xacro (robot description, xacro)
@@ -36,10 +36,10 @@
       </collision>
     </link>
-    <joint name="${prefix}plug_joint" type="fixed">
+    <joint name="${prefix}plug_rod_joint" type="fixed">
       <parent link="${prefix}plug_border"/>
-      <child link="${prefix}plug"/>
+      <child link="${prefix}plug_rod"/>
       <origin rpy="0.0 0.0 0.0" xyz="0.0 0.0 ${length_border/2.0+length_plug/2.0}"/>
     </joint>
-    <link name="${prefix}plug">
+    <link name="${prefix}plug_rod">
       <xacro:inertial_cylinder radius="${radius_plug}" length="${length_plug}" mass="${mass_plug}">
         <origin xyz="0 0 0" rpy="0 0 0"/>
@@ -59,8 +59,8 @@
     <!-- virtual reference frame -->
     <xacro:chargepal_virtual_joint
-      joint_name="${prefix}plug_ref_frame_joint"
+      joint_name="${prefix}plug_joint"
       type="fixed"
       parent="${prefix}plug_border"
-      child="${prefix}plug_reference_frame"
+      child="${prefix}plug"
       joint_axis_xyz="0 0 0"
       joint_origin_xyz="0 0 ${length_border/2.0}"
@@ -69,9 +69,9 @@
       joint_upper_limit="0"
     />
-    <xacro:chargepal_virtual_link link_name="${prefix}plug_reference_frame" />
-    <gazebo reference="handle">
+    <xacro:chargepal_virtual_link link_name="${prefix}plug" />
+    <gazebo reference="plug_border">
       <material>Gazebo/ZincYellow</material>
     </gazebo>
-    <gazebo reference="plug">
+    <gazebo reference="plug_rod">
       <material>Gazebo/ZincYellow</material>
     </gazebo>

File: urdf/tools/tdt_plug.urdf.xacro (robot description, xacro)
@@ -38,5 +38,5 @@
     <!-- virtual reference frame -->
     <xacro:chargepal_virtual_joint
-      joint_name="${prefix}plug_ref_frame_joint"
+      joint_name="${prefix}plug_joint"
       type="fixed"
       parent="${prefix}plug_root"
