Commit message: Add scaling for the plug meshes to test different plug-socket tolerances

File: _bullet_urdf_models/chargepal_testbed_tdt.urdf (robot description, URDF)
Before this commit: robot chargepal_testbed, 23 links, 22 joints
Links:
- link plug_root: geometry collision mesh filename=package://chargepal_tools/plugs/meshes/collision/tdt_plug_c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 scale=0.95 0.95 0.95; visual mesh filename=package://chargepal_tools/plugs/meshes/visual/tdt_plug_visu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 scale=0.95 0.95 0.95

File: urdf/tools/tdt_plug.urdf.xacro (robot description, xacro)
@@ -12,4 +12,5 @@
   <xacro:property name="plug_length" value="0.065" />
   <xacro:property name="plug_border_length" value="0.020" />
+  <xacro:property name="mesh_scale" value="0.95" />
   <xacro:macro name="tdt_plug" params="parent prefix">
     <joint name="${prefix}plug_root_joint" type="fixed">
@@ -22,5 +23,5 @@
         <origin xyz="0 0 0" rpy="0 0 0"/>
         <geometry>
-          <mesh filename="package://chargepal_tools/plugs/meshes/visual/tdt_plug_visual.obj"/>
+          <mesh filename="package://chargepal_tools/plugs/meshes/visual/tdt_plug_visual.obj" scale="${mesh_scale} ${mesh_scale} ${mesh_scale}"/>
         </geometry>
         <xacro:insert_block name="material_field_green" />
@@ -29,5 +30,5 @@
         <origin xyz="0 0 0" rpy="0 0 0"/>
         <geometry>
-          <mesh filename="package://chargepal_tools/plugs/meshes/collision/tdt_plug_collision.obj"/>
+          <mesh filename="package://chargepal_tools/plugs/meshes/collision/tdt_plug_collision.obj" scale="${mesh_scale} ${mesh_scale} ${mesh_scale}"/>
         </geometry>
       </collision>
