Commit message: Update plug scaling. Reduce clearance

File: _bullet_urdf_models/chargepal_testbed_cic.urdf (robot description, URDF)
Before this commit: robot chargepal_testbed, 23 links, 22 joints
Links:
- link plug_root: geometry collision mesh filename=package://chargepal_tools/plugs/meshes/collision/tdt_plug_c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 scale=0.99 0.99 0.99; visual mesh filename=package://chargepal_tools/plugs/meshes/visual/tdt_plug_visu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 scale=0.99 0.99 0.99

File: _bullet_urdf_models/chargepal_testbed_tdt.urdf (robot description, URDF)
Before this commit: robot chargepal_testbed, 23 links, 22 joints
Links:
- link plug_root: geometry collision mesh filename=package://chargepal_tools/plugs/meshes/collision/tdt_plug_c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 scale=0.99 0.99 0.99; visual mesh filename=package://chargepal_tools/plugs/meshes/visual/tdt_plug_visu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 scale=0.99 0.99 0.99

File: _bullet_urdf_models/ur10e_fix_plug.urdf (robot description, URDF)
Before this commit: robot chargepal_testbed, 20 links, 19 joints
Links:
- link plug_root: geometry collision mesh filename=package://chargepal_tools/plugs/meshes/collision/tdt_plug_c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 scale=0.99 0.99 0.99; visual mesh filename=package://chargepal_tools/plugs/meshes/visual/tdt_plug_visu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 scale=0.99 0.99 0.99

File: urdf/tools/tdt_plug.urdf.xacro (robot description, xacro)
@@ -12,5 +12,5 @@
   <xacro:property name="plug_length" value="0.065" />
   <xacro:property name="plug_border_length" value="0.020" />
-  <xacro:property name="mesh_scale" value="0.95" />
+  <xacro:property name="mesh_scale" value="0.99" />
   <xacro:macro name="tdt_plug" params="parent prefix">
     <joint name="${prefix}plug_root_joint" type="fixed">

Commit message: Relax tool clearance

File: _bullet_urdf_models/chargepal_testbed_cic.urdf (robot description, URDF)
Before this commit: robot chargepal_testbed, 23 links, 22 joints
Links:
- link plug_root: geometry collision mesh filename=package://chargepal_tools/plugs/meshes/collision/tdt_plug_c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 scale=0.98 0.98 0.98; visual mesh filename=package://chargepal_tools/plugs/meshes/visual/tdt_plug_visu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 scale=0.98 0.98 0.98

File: _bullet_urdf_models/chargepal_testbed_tdt.urdf (robot description, URDF)
Before this commit: robot chargepal_testbed, 23 links, 22 joints
Links:
- link plug_root: geometry collision mesh filename=package://chargepal_tools/plugs/meshes/collision/tdt_plug_c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 scale=0.98 0.98 0.98; visual mesh filename=package://chargepal_tools/plugs/meshes/visual/tdt_plug_visu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 scale=0.98 0.98 0.98

File: _bullet_urdf_models/ur10e_fix_plug.urdf (robot description, URDF)
Before this commit: robot chargepal_testbed, 20 links, 19 joints
Links:
- link plug_root: geometry collision mesh filename=package://chargepal_tools/plugs/meshes/collision/tdt_plug_c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 scale=0.98 0.98 0.98; visual mesh filename=package://chargepal_tools/plugs/meshes/visual/tdt_plug_visu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 scale=0.98 0.98 0.98

File: urdf/tools/tdt_plug.urdf.xacro (robot description, xacro)
@@ -12,5 +12,5 @@
   <xacro:property name="plug_length" value="0.065" />
   <xacro:property name="plug_border_length" value="0.020" />
-  <xacro:property name="mesh_scale" value="0.99" />
+  <xacro:property name="mesh_scale" value="0.98" />
   <xacro:macro name="tdt_plug" params="parent prefix">
     <joint name="${prefix}plug_root_joint" type="fixed">
