Commit message: Split robot and environment

File: _bullet_urdf_models/ur10e_ccs_type2.urdf (robot description, URDF)
Before this commit: robot chargepal_testbed, 23 links, 22 joints
Links:
- removed link arm_base
- removed link base_plate
- removed link table
Joints:
- removed joint baseplate_to_arm
- removed joint table_to_baseplate
- removed joint testbed_to_ur10e
- removed joint world_to_table
- added joint world_to_ur10e: type fixed, parent world, child base_link, origin xyz=0.0 0.0 0.0 rpy=0.0 0.0 3.14159

Commit message: Update plug scaling

File: _bullet_urdf_models/ur10e_ccs_type2.urdf (robot description, URDF)
Before this commit: robot chargepal_testbed, 20 links, 19 joints
Links:
- link plug_mounting: geometry collision mesh filename=package://chargepal_tools/plugs/meshes/collision/ccs_type2_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; collision mesh filename=package://chargepal_tools/plugs/meshes/collision/ccs_type2_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 scale=0.935 1.0 0.935

File: urdf/bringups/ur10e_ccs_type2.urdf.xacro (robot description, xacro)
@@ -75,5 +75,6 @@
   <!-- ############### FIX CCS TYPE 2 PLUG ################ -->
   <xacro:include filename="$(find chargepal_tools)/urdf/ccs_type2_plug.urdf.xacro" />
-  <xacro:ccs_type2_tool parent="${prefix}ft_sensor_wrench" prefix="${prefix}" collision_scale="1.0" />
+  <!-- collision scale upper limit 0.94 -->
+  <xacro:ccs_type2_tool parent="${prefix}ft_sensor_wrench" prefix="${prefix}" collision_scale="0.935" />
   <!-- ################ GAZEBO ################ -->
   <!-- Common -->

Commit message: Update scaling parameter of the plug

File: _bullet_urdf_models/ur10e_ccs_type2.urdf (robot description, URDF)
Before this commit: robot chargepal_testbed, 20 links, 19 joints
Links:
- link plug_mounting: geometry collision mesh filename=package://chargepal_tools/plugs/meshes/collision/ccs_type2_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; collision mesh filename=package://chargepal_tools/plugs/meshes/collision/ccs_type2_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 scale=0.92 1.0 0.92

File: urdf/bringups/ur10e_ccs_type2.urdf.xacro (robot description, xacro)
@@ -76,5 +76,5 @@
   <xacro:include filename="$(find chargepal_tools)/urdf/ccs_type2_plug.urdf.xacro" />
   <!-- collision scale upper limit 0.94 -->
-  <xacro:ccs_type2_tool parent="${prefix}ft_sensor_wrench" prefix="${prefix}" collision_scale="0.935" />
+  <xacro:ccs_type2_tool parent="${prefix}ft_sensor_wrench" prefix="${prefix}" collision_scale="0.92" />
   <!-- ################ GAZEBO ################ -->
   <!-- Common -->
