Commit message: Clean up and remove old unused models

File: _bullet_urdf_models/ccs_socket_wall.urdf (robot description, URDF)
Before this commit: robot adapter_station_square_socket, 7 links, 6 joints
Joints:
- removed joint world_joint
- added joint socket_base_joint: type fixed, parent world, child socket_base, origin xyz=0 0 0.5 rpy=1.5707963267948966 0 -1.5707963267948966

File: _bullet_urdf_models/cpm_fix_rod_30.urdf (robot description, URDF)
Before this commit: robot cpm_fix_rod_30, 23 links, 22 joints
Links:
- removed link plug
- added link plug_lip, mass 0.0
- added link plug_mounting, mass 0.0
- added link plug_tip, mass 0.0
Joints:
- removed joint plug_joint
- added joint plug_lip_joint: type fixed, parent rod, child plug_lip, origin xyz=0 0 -0.015000000000000003 rpy=0 0 0, axis 0 0 0
- added joint plug_mounting_joint: type fixed, parent rod, child plug_mounting, origin xyz=0 0 -0.035 rpy=0 0 0, axis 0 0 0
- added joint plug_tip_joint: type fixed, parent rod, child plug_tip, origin xyz=0 0 0.035 rpy=0 0 0, axis 0 0 0

File: _bullet_urdf_models/cpm_fix_rod_32d5.urdf (robot description, URDF)
Before this commit: robot cpm_fix_rod_30, 23 links, 22 joints
Links:
- removed link plug
- added link plug_lip, mass 0.0
- added link plug_mounting, mass 0.0
- added link plug_tip, mass 0.0
Joints:
- removed joint plug_joint
- added joint plug_lip_joint: type fixed, parent rod, child plug_lip, origin xyz=0 0 -0.015000000000000003 rpy=0 0 0, axis 0 0 0
- added joint plug_mounting_joint: type fixed, parent rod, child plug_mounting, origin xyz=0 0 -0.035 rpy=0 0 0, axis 0 0 0
- added joint plug_tip_joint: type fixed, parent rod, child plug_tip, origin xyz=0 0 0.035 rpy=0 0 0, axis 0 0 0

File: _bullet_urdf_models/cpm_fix_rod_34.urdf (robot description, URDF)
Before this commit: robot cpm_fix_rod_30, 23 links, 22 joints
Links:
- removed link plug
- added link plug_lip, mass 0.0
- added link plug_mounting, mass 0.0
- added link plug_tip, mass 0.0
Joints:
- removed joint plug_joint
- added joint plug_lip_joint: type fixed, parent rod, child plug_lip, origin xyz=0 0 -0.015000000000000003 rpy=0 0 0, axis 0 0 0
- added joint plug_mounting_joint: type fixed, parent rod, child plug_mounting, origin xyz=0 0 -0.035 rpy=0 0 0, axis 0 0 0
- added joint plug_tip_joint: type fixed, parent rod, child plug_tip, origin xyz=0 0 0.035 rpy=0 0 0, axis 0 0 0

File: _bullet_urdf_models/cpm_fix_rod_34d5.urdf (robot description, URDF)
Before this commit: robot cpm_fix_rod_30, 23 links, 22 joints
Links:
- removed link plug
- added link plug_lip, mass 0.0
- added link plug_mounting, mass 0.0
- added link plug_tip, mass 0.0
Joints:
- removed joint plug_joint
- added joint plug_lip_joint: type fixed, parent rod, child plug_lip, origin xyz=0 0 -0.015000000000000003 rpy=0 0 0, axis 0 0 0
- added joint plug_mounting_joint: type fixed, parent rod, child plug_mounting, origin xyz=0 0 -0.035 rpy=0 0 0, axis 0 0 0
- added joint plug_tip_joint: type fixed, parent rod, child plug_tip, origin xyz=0 0 0.035 rpy=0 0 0, axis 0 0 0

File: _bullet_urdf_models/primitive_chargepal_with_fix_plug.urdf (robot description, URDF)
Before this commit: robot primitive_chargepal_with_fix_plug, 24 links, 23 joints
Links:
- removed link plug
- removed link plug_border
- removed link plug_rod
- added link plug_lip, mass 0.0
- added link plug_mounting, mass 0.2; collision mesh filename=package://chargepal_tools/plugs/meshes/collision/tdt_plug_c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 scale=0.98 0.98 1.0; visual mesh filename=package://chargepal_tools/plugs/meshes/visual/tdt_plug_visu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 scale=0.98 0.98 1.0
- added link plug_tip, mass 0.0
Joints:
- removed joint plug_border_joint
- removed joint plug_joint
- removed joint plug_rod_joint
- added joint plug_lip_joint: type fixed, parent plug_mounting, child plug_lip, origin xyz=0 0 0.02 rpy=0 0 0, axis 0 0 0
- added joint plug_mounting_joint: type fixed, parent ft_sensor_wrench, child plug_mounting, origin xyz=0.0 0.0 0.0 rpy=0.0 0.0 0.0
- added joint plug_tip_joint: type fixed, parent plug_mounting, child plug_tip, origin xyz=0 0 0.065 rpy=0 0 0, axis 0 0 0

File: _bullet_urdf_models/ur10e_ccs_type2.urdf (robot description, URDF)
Before this commit: robot chargepal_testbed, 20 links, 19 joints
Links:
- added link plug_lip, mass 0.0
Joints:
- removed joint handle_joint
- removed joint plug_joint
- added joint plug_lip_joint: type fixed, parent plug_mounting, child plug_lip, origin xyz=0 0 0.05 rpy=0 0 0, axis 0 0 0
- added joint plug_mounting_joint: type fixed, parent ft_sensor_wrench, child plug_mounting, origin xyz=0.0 0.0 0.0 rpy=0 0 0
- added joint plug_tip_joint: type fixed, parent plug_mounting, child plug_tip, origin xyz=0 0 0.085 rpy=0 0 0, axis 0 0 0

File: _bullet_urdf_models/ur10e_fix_plug.urdf (robot description, URDF)
Before this commit: robot chargepal_testbed, 20 links, 19 joints
Links:
- removed link plug
- removed link plug_root
- added link plug_lip, mass 0.0
- added link plug_mounting, mass 0.2; collision mesh filename=package://chargepal_tools/plugs/meshes/collision/tdt_plug_c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 scale=0.98 0.98 1.0; visual mesh filename=package://chargepal_tools/plugs/meshes/visual/tdt_plug_visu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 scale=0.98 0.98 1.0
- added link plug_tip, mass 0.0
Joints:
- removed joint plug_joint
- removed joint plug_root_joint
- added joint plug_lip_joint: type fixed, parent plug_mounting, child plug_lip, origin xyz=0 0 0.02 rpy=0 0 0, axis 0 0 0
- added joint plug_mounting_joint: type fixed, parent ft_sensor_wrench, child plug_mounting, origin xyz=0.0 0.0 0.0 rpy=0.0 0.0 0.0
- added joint plug_tip_joint: type fixed, parent plug_mounting, child plug_tip, origin xyz=0 0 0.065 rpy=0 0 0, axis 0 0 0

File: urdf/robots/cpm_fix_rod_30.urdf.xacro (robot description, xacro)
@@ -4,5 +4,5 @@
   <xacro:include filename="$(find chargepal_description)/urdf/utils/prefix.urdf.xacro" />
   <!-- Include rod tool xacro-->
-  <xacro:include filename="$(find chargepal_description)/urdf/bringups/cpm_fix_rod_macro.urdf.xacro" />
+  <xacro:include filename="$(find chargepal_description)/urdf/robots/cpm_fix_rod_macro.urdf.xacro" />
   <xacro:generic_chargepal_model prefix="${prefix}" rod_diameter="30" />
 </robot>

File: urdf/robots/cpm_fix_rod_32d5.urdf.xacro (robot description, xacro)
@@ -4,5 +4,5 @@
   <xacro:include filename="$(find chargepal_description)/urdf/utils/prefix.urdf.xacro" />
   <!-- Include rod tool xacro-->
-  <xacro:include filename="$(find chargepal_description)/urdf/bringups/cpm_fix_rod_macro.urdf.xacro" />
-  <xacro:generic_chargepal_model prefix="${prefix}" rod_diameter="34.5" />
+  <xacro:include filename="$(find chargepal_description)/urdf/robots/cpm_fix_rod_macro.urdf.xacro" />
+  <xacro:generic_chargepal_model prefix="${prefix}" rod_diameter="32.5" />
 </robot>

File: urdf/robots/cpm_fix_rod_34.urdf.xacro (robot description, xacro)
@@ -4,5 +4,5 @@
   <xacro:include filename="$(find chargepal_description)/urdf/utils/prefix.urdf.xacro" />
   <!-- Include rod tool xacro-->
-  <xacro:include filename="$(find chargepal_description)/urdf/bringups/cpm_fix_rod_macro.urdf.xacro" />
-  <xacro:generic_chargepal_model prefix="${prefix}" rod_diameter="32.5" />
+  <xacro:include filename="$(find chargepal_description)/urdf/robots/cpm_fix_rod_macro.urdf.xacro" />
+  <xacro:generic_chargepal_model prefix="${prefix}" rod_diameter="34" />
 </robot>

File: urdf/robots/cpm_fix_rod_34d5.urdf.xacro (robot description, xacro)
@@ -4,5 +4,5 @@
   <xacro:include filename="$(find chargepal_description)/urdf/utils/prefix.urdf.xacro" />
   <!-- Include rod tool xacro-->
-  <xacro:include filename="$(find chargepal_description)/urdf/bringups/cpm_fix_rod_macro.urdf.xacro" />
-  <xacro:generic_chargepal_model prefix="${prefix}" rod_diameter="34" />
+  <xacro:include filename="$(find chargepal_description)/urdf/robots/cpm_fix_rod_macro.urdf.xacro" />
+  <xacro:generic_chargepal_model prefix="${prefix}" rod_diameter="34.5" />
 </robot>

File: urdf/robots/cpm_fix_rod_macro.urdf.xacro (robot description, xacro)
@@ -77,6 +77,6 @@
     </joint>
     <!-- ############### FIX PLUG ################ -->
-    <xacro:include filename="$(find chargepal_tools)/urdf/rod.urdf.xacro" />
-    <xacro:rod_tool parent="${prefix}ft_sensor_wrench" prefix="${prefix}" diameter="${rod_diameter}" />
+    <xacro:include filename="$(find chargepal_tools)/urdf/rod_plug.urdf.xacro" />
+    <xacro:rod_plug_tool parent="${prefix}ft_sensor_wrench" prefix="${prefix}" diameter="${rod_diameter}" />
     <!-- ################ GAZEBO ################ -->
     <!-- Common -->

File: urdf/robots/primitive_chargepal_with_fix_plug.urdf.xacro (robot description, xacro)
@@ -1,4 +1,4 @@
 <?xml version="1.0"?>
-<robot xmlns:xacro="http://ros.org/wiki/xacro" name="chargepal_testbed">
+<robot xmlns:xacro="http://ros.org/wiki/xacro" name="primitive_chargepal_with_fix_plug">
   <!-- Macros -->
   <xacro:include filename="$(find chargepal_description)/urdf/utils/chargepal_common.urdf.xacro" />
@@ -7,16 +7,16 @@
   <!-- Resolve prefix variable (useful for multi robot) -->
   <xacro:include filename="$(find chargepal_description)/urdf/utils/prefix.urdf.xacro" />
-  <!-- ############### Table ################ -->
-  <xacro:include filename="$(find chargepal_description)/urdf/environment/testbed_table_cic.urdf.xacro"/>
+  <!-- ############### PLATFORM ################ -->
+  <xacro:include filename="$(find chargepal_description)/urdf/mobile_platform/primitive_mobile_platform.urdf.xacro"/>
   <!-- platform arm joint -->
-  <joint name="${prefix}testbed_to_ur10e" type="fixed">
-    <parent link="${prefix}arm_base" />
+  <joint name="${prefix}platform_ur10e_joint" type="fixed">
+    <parent link="${prefix}tower_link" />
     <child link="${prefix}base_link" />
-    <origin xyz="0.0 0.0 0.0" rpy="0.0 0.0 ${-0.5*M_PI}" />
+    <origin xyz="0.0 0.0 ${tower_height/2}" rpy="0.0 0.0 ${0.5*M_PI}" />
   </joint>
   <!-- ############### UR10e ARM ################ -->
   <xacro:include filename="$(find ur_description)/urdf/inc/ur10e_macro.xacro"/>
   <!-- Arguments to load UR10e arm macro -->
-  <xacro:arg name="joint_limit_params" default="$(find ur_description)/config/ur10e/joint_limits.yaml"/>
+  <xacro:arg name="joint_limit_params" default="$(find chargepal_description)/config/ur10e/joint_limits.yaml"/>
   <xacro:arg name="physical_params" default="$(find ur_description)/config/ur10e/physical_parameters.yaml"/>
   <xacro:arg name="kinematics_params" default="$(find ur_description)/config/ur10e/default_kinematics.yaml"/>
@@ -75,7 +75,7 @@
     <origin xyz="0.0 0.0 0.0" rpy="0.0 0.0 0.0" />
   </joint>
-  <!-- ############### FIX ROD ################ -->
-  <xacro:include filename="$(find chargepal_description)/urdf/tools/tdt_plug.urdf.xacro" />
-  <xacro:tdt_plug parent="${prefix}ft_sensor_wrench" prefix="${prefix}" />
+  <!-- ############### FIX PLUG ################ -->
+  <xacro:include filename="$(find chargepal_tools)/urdf/tdt_plug.urdf.xacro" />
+  <xacro:tdt_plug parent="${prefix}ft_sensor_wrench" prefix="${prefix}" mesh_scale="0.98"/>
   <!-- ################ GAZEBO ################ -->
   <!-- Common -->

File: urdf/robots/ur10e_fix_plug.urdf.xacro (robot description, xacro)
@@ -74,6 +74,6 @@
   </joint>
   <!-- ############### FIX ROD ################ -->
-  <xacro:include filename="$(find chargepal_description)/urdf/tools/tdt_plug.urdf.xacro" />
-  <xacro:tdt_plug parent="${prefix}ft_sensor_wrench" prefix="${prefix}" />
+  <xacro:include filename="$(find chargepal_tools)/urdf/tdt_plug.urdf.xacro" />
+  <xacro:tdt_plug parent="${prefix}ft_sensor_wrench" prefix="${prefix}" mesh_scale="0.98"/>
   <!-- ################ GAZEBO ################ -->
   <!-- Common -->
